File: hardware/bringup-board/bringup-board.kicad_pcb (KiCad board)
At the start: 2 copper layers, 115 x 98 mm, 50 parts, among them J1 FLASH, J2 CPU_JTAG, J3 SPI_I2C_GPIO, J4 PWM_PDM, J5 UART0, J6 UART1, J7 USB_B_Micro, J8 5V, SW1 RESET, U2 LD39015M33R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

Commit message: push latest updates
Signed-off-by: gatecat <gatecat@ds0.me>
Parts:
- C4: moved to B.Cu
- moved J4 57.0 mm to (106.0, 117.0)
- moved J3 56.0 mm to (50.0, 117.0)
- moved C4 7.25 mm to (109.0, 91.8)
- moved RN1 7.01 mm to (142.5, 84.8)
- moved RN2 7.01 mm to (142.5, 90.8)
- moved C2 4.92 mm to (69.5, 60.7)
- turned C6 to -90 degrees
Connections:
- J4 pad 10: /PWM6_PWM -> /PWM2_DIR
- J4 pad 11: /PWM1_DIR -> /PWM3_DIR
- J4 pad 12: /PWM6_DIR -> /PWM2_PWM
- J4 pad 13: /PWM1_STOP -> /PWM3_PWM
- J4 pad 14: /PWM6_STOP -> /PWM4_PWM
- J4 pad 15: /PWM2_PWM -> /PWM3_STOP
- J4 pad 16: /PWM7_PWM -> /PWM5_PWM
- J4 pad 17: /PWM2_DIR -> /PWM4_DIR
- J4 pad 18: /PWM7_DIR -> /PWM4_STOP
- J4 pad 19: /PWM2_STOP -> /PWM5_STOP
- J4 pad 20: /PWM7_STOP -> /PWM5_DIR
- J4 pad 21: /PWM3_PWM -> /PWM6_PWM
- J4 pad 22: /PWM8_PWM -> /PWM7_PWM
- J4 pad 23: /PWM3_DIR -> /PWM6_DIR
- J4 pad 24: /PWM8_DIR -> /PWM6_STOP
- J4 pad 25: /PWM3_STOP -> /PWM7_DIR
- J4 pad 26: /PWM8_STOP -> /PWM8_PWM
- J4 pad 27: /PWM4_PWM -> /PWM7_STOP
- J4 pad 28: /PWM9_PWM -> /PWM8_STOP
- J4 pad 29: /PWM4_DIR -> /PWM8_DIR
- J4 pad 31: /PWM4_STOP -> /PWM9_PWM
- J4 pad 4: /PWM5_STOP -> /PWM1_PWM
- J4 pad 6: /PWM5_DIR -> /PWM0_STOP
- J4 pad 7: /PWM0_STOP -> /PWM1_DIR
- J4 pad 8: /PWM5_PWM -> /PWM1_STOP
- J4 pad 9: /PWM1_PWM -> /PWM2_STOP
Routing:
- net +3V3: track 0.00 -> 499.1 mm, vias 0 -> 11
- net +1V5: track 0.00 -> 117.0 mm
- net /GPIO0_2: track 0.00 -> 116.5 mm, vias 0 -> 2
- net /GPIO0_7: track 0.00 -> 114.5 mm, vias 0 -> 2
- net /GPIO0_6: track 0.00 -> 113.8 mm, vias 0 -> 2
- net /GPIO0_1: track 0.00 -> 112.2 mm, vias 0 -> 3
- net /GPIO0_5: track 0.00 -> 110.2 mm, vias 0 -> 3
- net /GPIO0_3: track 0.00 -> 109.9 mm, vias 0 -> 3
- net /GPIO0_4: track 0.00 -> 105.4 mm, vias 0 -> 3
- net /GPIO1_7: track 0.00 -> 105.1 mm
- net /GPIO0_0: track 0.00 -> 103.9 mm, vias 0 -> 3
- net /GPIO1_4: track 0.00 -> 103.6 mm, vias 0 -> 1
- net /GPIO1_3: track 0.00 -> 103.1 mm, vias 0 -> 2
- net /GPIO1_5: track 0.00 -> 102.5 mm
- net /GPIO1_6: track 0.00 -> 101.6 mm
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- added copper zone on B.Cu, net GND
- added copper zone on F.Cu, net GND
- added copper zone on In1.Cu, net GND
- added copper zone on In2.Cu, net GND
Other:
- copper layers 2 -> 4
