File: hardware/bringup-board/bringup-board.kicad_sch (KiCad schematic)
At the start: 50 parts, among them J1 FLASH, J2 CPU_JTAG, J3 SPI_I2C_GPIO, J4 PWM_PDM, J5 UART0, J6 UART1, J7 USB_B_Micro, J8 5V, SW1 RESET, U2 LD39015M33R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

Commit message: outline pcb placement
Signed-off-by: gatecat <gatecat@ds0.me>
Parts:
- C1, C10, C11, C2, C3, C4, C5, C6, C7, C8, C9: footprint (none) -> Capacitor_SMD:C_0603_1608Metric
- D1, D10, D2, D3, D4, D5, D6, D7, D8, D9: footprint (none) -> LED_SMD:LED_0805_2012Metric
- J1: footprint (none) -> Connector_PinHeader_2.54mm:PinHeader_1x08_P2.54mm_Vertical
- J2: footprint (none) -> Connector_IDC:IDC-Header_2x05_P2.54mm_Vertical
- J3, J4: footprint (none) -> Connector_PinHeader_2.54mm:PinHeader_2x20_P2.54mm_Vertical
- J5, J6: footprint (none) -> Connector_PinHeader_2.54mm:PinHeader_1x04_P2.54mm_Vertical
- J7: footprint (none) -> Connector_USB:USB_Micro-B_Molex-105017-0001
- J8, JP1, JP2, JP3: footprint (none) -> Connector_PinHeader_2.54mm:PinHeader_1x02_P2.54mm_Vertical
- R1, R2, R3, R4, R5, R6, R7, R8, R9: footprint (none) -> Resistor_SMD:R_0603_1608Metric
- RN1, RN2: footprint (none) -> Resistor_SMD:R_Array_Convex_4x0402
- SW1: footprint (none) -> Button_Switch_SMD:SW_SPST_B3S-1000
- U1: footprint (none) -> bringup_board_parts:145-PRS15024-12
- U4: value ~ -> SN74CB3Q3244DBQR; footprint (none) -> Package_SO:SSOP-20_3.9x8.7mm_P0.635mm
Changed lines of the file:
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@@
 			)
 		)
-		(property "Footprint" ""
+		(property "Footprint" "Button_Switch_SMD:SW_SPST_B3S-1000"
 			(at 46.99 124.46 0)
 			(effects
@@
 			)
 		)
-		(property "Footprint" ""
+		(property "Footprint" "Connector_PinHeader_2.54mm:PinHeader_1x04_P2.54mm_Vertical"
 			(at 297.18 198.12 0)
 			(effects
@@
 			)
 		)
-		(property "Footprint" ""
+		(property "Footprint" "Connector_PinHeader_2.54mm:PinHeader_2x20_P2.54mm_Vertical"
 			(at 294.64 161.29 0)
 			(effects
@@
 			)
 		)
-		(property "Footprint" ""
+		(property "Footprint" "Capacitor_SMD:C_0603_1608Metric"
 			(at 93.98 57.15 0)
 			(effects
@@
 			)
 		)
-		(property "Footprint" ""
+		(property "Footprint" "Connector_PinHeader_2.54mm:PinHeader_2x20_P2.54mm_Vertical"
 			(at 294.64 99.06 0)
 			(effects
@@
 			)
 		)
-		(property "Footprint" ""
+		(property "Footprint" "Capacitor_SMD:C_0603_1608Metric"
 			(at 20.32 31.75 0)
 			(effects
@@
 			)
 		)
-		(property "Footprint" ""
+		(property "Footprint" "LED_SMD:LED_0805_2012Metric"
 			(at 259.08 228.6 0)
 			(effects
@@
 			)
 		)
-		(property "Footprint" ""
+		(property "Footprint" "Resistor_SMD:R_Array_Convex_4x0402"
 			(at 242.57 273.685 90)
 			(effects
@@
 			)
 		)
-		(property "Footprint" ""
+		(property "Footprint" "Resistor_SMD:R_0603_1608Metric"
 			(at 242.57 236.22 0)
 			(effects
@@
 			)
 		)
-		(property "Footprint" ""
+		(property "Footprint" "Resistor_SMD:R_0603_1608Metric"
 			(at 267.97 209.55 0)
 			(effects
@@
 			)
 		)
-		(property "Footprint" ""
+		(property "Footprint" "Connector_PinHeader_2.54mm:PinHeader_1x04_P2.54mm_Vertical"
 			(at 297.18 213.36 0)
 			(effects
@@
 			)
 		)
-		(property "Footprint" ""
+		(property "Footprint" "Resistor_SMD:R_0603_1608Metric"
 			(at 267.97 194.31 0)
 			(effects
@@
 			)
 		)
-		(property "Footprint" ""
+		(property "Footprint" "LED_SMD:LED_0805_2012Metric"
 			(at 259.08 261.62 0)
 			(effects
@@
 			)
 		)
-		(property "Footprint" ""
+		(property "Footprint" "Connector_PinHeader_2.54mm:PinHeader_1x02_P2.54mm_Vertical"
 			(at 55.88 24.13 0)
 			(effects
@@
 			)
 		)
-		(property "Footprint" ""
+		(property "Footprint" "Resistor_SMD:R_0603_1608Metric"
 			(at 52.07 110.49 0)
 			(effects
@@
 			)
 		)
-		(property "Footprint" ""
+		(property "Footprint" "LED_SMD:LED_0805_2012Metric"
 			(at 259.08 248.92 0)
 			(effects
@@
 			)
 		)
-		(property "Footprint" ""
+		(property "Footprint" "Resistor_SMD:R_0603_1608Metric"
 			(at 220.98 48.26 0)
 			(effects
@@
 			)
 		)
-		(property "Footprint" ""
+		(property "Footprint" "Resistor_SMD:R_0603_1608Metric"
 			(at 242.57 228.6 0)
 			(effects
@@
 			)
 		)
-		(property "Footprint" ""
+		(property "Footprint" "Capacitor_SMD:C_0603_1608Metric"
 			(at 20.32 59.69 0)
 			(effects
@@
 			)
 		)
-		(property "Footprint" ""
+		(property "Footprint" "LED_SMD:LED_0805_2012Metric"
 			(at 259.08 269.24 0)
 			(effects
@@
 			)
 		)
-		(property "Footprint" ""
+		(property "Footprint" "bringup_board_parts:145-PRS15024-12"
 			(at 142.24 256.54 0)
 			(effects
@@
 			)
 		)
-		(property "Footprint" ""
+		(property "Footprint" "Connector_PinHeader_2.54mm:PinHeader_1x02_P2.54mm_Vertical"
 			(at 48.26 91.44 0)
 			(effects
@@
 			)
 		)
-		(property "Footprint" ""
+		(property "Footprint" "Connector_USB:USB_Micro-B_Molex-105017-0001"
 			(at 30.48 224.79 0)
 			(effects
@@
 			)
 		)
-		(property "Footprint" ""
+		(property "Footprint" "Capacitor_SMD:C_0603_1608Metric"
 			(at 46.99 59.69 0)
 			(effects
@@
 			)
 		)
-		(property "Footprint" ""
+		(property "Footprint" "Resistor_SMD:R_0603_1608Metric"
 			(at 68.58 185.42 0)
 			(effects
@@
 			)
 		)
-		(property "Footprint" ""
+		(property "Footprint" "Resistor_SMD:R_0603_1608Metric"
 			(at 68.58 160.02 0)
 			(effects
@@
 			)
 		)
-		(property "Footprint" ""
+		(property "Footprint" "Resistor_SMD:R_Array_Convex_4x0402"
 			(at 242.57 241.935 90)
 			(effects
@@
 			)
 		)
-		(property "Footprint" ""
+		(property "Footprint" "LED_SMD:LED_0805_2012Metric"
 			(at 259.08 246.38 0)
 			(effects
@@
 			)
 		)
-		(property "Footprint" ""
+		(property "Footprint" "LED_SMD:LED_0805_2012Metric"
 			(at 259.08 266.7 0)
 			(effects
@@
 			)
 		)
-		(property "Footprint" ""
+		(property "Footprint" "Capacitor_SMD:C_0603_1608Metric"
 			(at 86.36 57.15 0)
 			(effects
@@
 			)
 		)
-		(property "Footprint" ""
+		(property "Footprint" "Capacitor_SMD:C_0603_1608Metric"
 			(at 46.99 31.75 0)
 			(effects
@@
 			)
 		)
-		(property "Footprint" ""
+		(property "Footprint" "Capacitor_SMD:C_0603_1608Metric"
 			(at 102.87 41.91 0)
 			(effects
@@
 			)
 		)
-		(property "Footprint" ""
+		(property "Footprint" "Connector_PinHeader_2.54mm:PinHeader_1x08_P2.54mm_Vertical"
 			(at 360.68 33.02 0)
 			(effects
@@
 			)
 		)
-		(property "Footprint" ""
+		(property "Footprint" "LED_SMD:LED_0805_2012Metric"
 			(at 259.08 254 0)
 			(effects
@@
 			)
 		)
-		(property "Footprint" ""
+		(property "Footprint" "Capacitor_SMD:C_0603_1608Metric"
 			(at 95.25 41.91 0)
 			(effects
@@
 			)
 		)
-		(property "Footprint" ""
+		(property "Footprint" "Resistor_SMD:R_0603_1608Metric"
 			(at 273.05 24.13 0)
 			(effects
@@
 			)
 		)
-		(property "Footprint" ""
+		(property "Footprint" "Capacitor_SMD:C_0603_1608Metric"
 			(at 78.74 57.15 0)
 			(effects
@@
 			)
 		)
-		(property "Footprint" ""
+		(property "Footprint" "LED_SMD:LED_0805_2012Metric"
 			(at 259.08 236.22 0)
 			(effects
@@
 			)
 		)
-		(property "Value" "~"
+		(property "Value" "SN74CB3Q3244DBQR"
 			(at 236.22 13.97 0)
 			(effects
@@
 			)
 		)
-		(property "Footprint" ""
+		(property "Footprint" "Package_SO:SSOP-20_3.9x8.7mm_P0.635mm"
 			(at 236.22 55.88 0)
 			(effects
@@
 			)
 		)
-		(property "Footprint" ""
+		(property "Footprint" "Connector_PinHeader_2.54mm:PinHeader_1x02_P2.54mm_Vertical"
 			(at 55.88 52.07 0)
 			(effects
@@
 			)
 		)
-		(property "Footprint" ""
+		(property "Footprint" "LED_SMD:LED_0805_2012Metric"
 			(at 259.08 264.16 0)
 			(effects
@@
 			)
 		)
-		(property "Footprint" ""
+		(property "Footprint" "LED_SMD:LED_0805_2012Metric"
 			(at 259.08 251.46 0)
 			(effects
@@
 			)
 		)
-		(property "Footprint" ""
+		(property "Footprint" "Capacitor_SMD:C_0603_1608Metric"
 			(at 303.53 20.32 0)
 			(effects
@@
 			)
 		)
-		(property "Footprint" ""
+		(property "Footprint" "Capacitor_SMD:C_0603_1608Metric"
 			(at 24.13 82.55 0)
 			(effects
@@
 			)
 		)
-		(property "Footprint" ""
+		(property "Footprint" "Connector_IDC:IDC-Header_2x05_P2.54mm_Vertical"
 			(at 52.07 173.99 0)
 			(effects
@@
 			)
 		)
-		(property "Footprint" ""
+		(property "Footprint" "Connector_PinHeader_2.54mm:PinHeader_1x02_P2.54mm_Vertical"
 			(at 50.8 224.79 0)
 			(effects

Commit message: push latest updates
Signed-off-by: gatecat <gatecat@ds0.me>
Connections:
- net PWM0_STOP: now also J4.6 (Pin_6); no longer J4.7 (Pin_7)
- net PWM1_DIR: now also J4.7 (Pin_7); no longer J4.11 (Pin_11)
- net PWM1_PWM: now also J4.4 (Pin_4); no longer J4.9 (Pin_9)
- net PWM1_STOP: now also J4.8 (Pin_8); no longer J4.13 (Pin_13)
- net PWM2_DIR: now also J4.10 (Pin_10); no longer J4.17 (Pin_17)
- net PWM2_PWM: now also J4.12 (Pin_12); no longer J4.15 (Pin_15)
- net PWM2_STOP: now also J4.9 (Pin_9); no longer J4.19 (Pin_19)
- net PWM3_DIR: now also J4.11 (Pin_11); no longer J4.23 (Pin_23)
- net PWM3_PWM: now also J4.13 (Pin_13); no longer J4.21 (Pin_21)
- net PWM3_STOP: now also J4.15 (Pin_15); no longer J4.25 (Pin_25)
- net PWM4_DIR: now also J4.17 (Pin_17); no longer J4.29 (Pin_29)
- net PWM4_PWM: now also J4.14 (Pin_14); no longer J4.27 (Pin_27)
- net PWM4_STOP: now also J4.18 (Pin_18); no longer J4.31 (Pin_31)
- net PWM5_DIR: now also J4.20 (Pin_20); no longer J4.6 (Pin_6)
- net PWM5_PWM: now also J4.16 (Pin_16); no longer J4.8 (Pin_8)
- net PWM5_STOP: now also J4.19 (Pin_19); no longer J4.4 (Pin_4)
- net PWM6_DIR: now also J4.23 (Pin_23); no longer J4.12 (Pin_12)
- net PWM6_PWM: now also J4.21 (Pin_21); no longer J4.10 (Pin_10)
- net PWM6_STOP: now also J4.24 (Pin_24); no longer J4.14 (Pin_14)
- net PWM7_DIR: now also J4.25 (Pin_25); no longer J4.18 (Pin_18)
- net PWM7_PWM: now also J4.22 (Pin_22); no longer J4.16 (Pin_16)
- net PWM7_STOP: now also J4.27 (Pin_27); no longer J4.20 (Pin_20)
- net PWM8_DIR: now also J4.29 (Pin_29); no longer J4.24 (Pin_24)
- net PWM8_PWM: now also J4.26 (Pin_26); no longer J4.22 (Pin_22)
- net PWM8_STOP: now also J4.28 (Pin_28); no longer J4.26 (Pin_26)
- net PWM9_PWM: now also J4.31 (Pin_31); no longer J4.28 (Pin_28)
Changed lines of the file:
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@@
 		)
 	)
-	(label "PWM5_STOP"
+	(label "PWM1_PWM"
 		(at 318.77 140.97 180)
 		(fields_autoplaced yes)
@@
 		)
 	)
-	(label "PWM5_PWM"
+	(label "PWM1_STOP"
 		(at 318.77 146.05 180)
 		(fields_autoplaced yes)
@@
 		)
 	)
-	(label "PWM2_STOP"
+	(label "PWM5_STOP"
 		(at 273.05 161.29 0)
 		(fields_autoplaced yes)
@@
 		)
 	)
-	(label "PWM6_PWM"
+	(label "PWM2_DIR"
 		(at 318.77 148.59 180)
 		(fields_autoplaced yes)
@@
 		)
 	)
-	(label "PWM1_DIR"
+	(label "PWM3_DIR"
 		(at 273.05 151.13 0)
 		(fields_autoplaced yes)
@@
 		)
 	)
-	(label "PWM3_STOP"
+	(label "PWM7_DIR"
 		(at 273.05 168.91 0)
 		(fields_autoplaced yes)
@@
 		)
 	)
-	(label "PWM4_DIR"
+	(label "PWM8_DIR"
 		(at 273.05 173.99 0)
 		(fields_autoplaced yes)
@@
 		)
 	)
-	(label "PWM1_PWM"
+	(label "PWM2_STOP"
 		(at 273.05 148.59 0)
 		(fields_autoplaced yes)
@@
 		)
 	)
-	(label "PWM2_DIR"
+	(label "PWM4_DIR"
 		(at 273.05 158.75 0)
 		(fields_autoplaced yes)
@@
 		)
 	)
-	(label "PWM5_DIR"
+	(label "PWM0_STOP"
 		(at 318.77 143.51 180)
 		(fields_autoplaced yes)
@@
 		)
 	)
-	(label "PWM3_DIR"
+	(label "PWM6_DIR"
 		(at 273.05 166.37 0)
 		(fields_autoplaced yes)
@@
 		)
 	)
-	(label "PWM7_PWM"
+	(label "PWM5_PWM"
 		(at 318.77 156.21 180)
 		(fields_autoplaced yes)
@@
 		)
 	)
-	(label "PWM4_PWM"
+	(label "PWM7_STOP"
 		(at 273.05 171.45 0)
 		(fields_autoplaced yes)
@@
 		)
 	)
-	(label "PWM8_PWM"
+	(label "PWM7_PWM"
 		(at 318.77 163.83 180)
 		(fields_autoplaced yes)
@@
 		)
 	)
-	(label "PWM8_STOP"
+	(label "PWM8_PWM"
 		(at 318.77 168.91 180)
 		(fields_autoplaced yes)
@@
 		)
 	)
-	(label "PWM6_STOP"
+	(label "PWM4_PWM"
 		(at 318.77 153.67 180)
 		(fields_autoplaced yes)
@@
 		)
 	)
-	(label "PWM7_DIR"
+	(label "PWM4_STOP"
 		(at 318.77 158.75 180)
 		(fields_autoplaced yes)
@@
 		)
 	)
-	(label "PWM4_STOP"
+	(label "PWM9_PWM"
 		(at 273.05 176.53 0)
 		(fields_autoplaced yes)
@@
 		)
 	)
-	(label "PWM0_STOP"
+	(label "PWM1_DIR"
 		(at 273.05 146.05 0)
 		(fields_autoplaced yes)
@@
 		)
 	)
-	(label "PWM1_STOP"
+	(label "PWM3_PWM"
 		(at 273.05 153.67 0)
 		(fields_autoplaced yes)
@@
 		)
 	)
-	(label "PWM8_DIR"
+	(label "PWM6_STOP"
 		(at 318.77 166.37 180)
 		(fields_autoplaced yes)
@@
 		)
 	)
-	(label "PWM2_PWM"
+	(label "PWM3_STOP"
 		(at 273.05 156.21 0)
 		(fields_autoplaced yes)
@@
 		)
 	)
-	(label "PWM3_PWM"
+	(label "PWM6_PWM"
 		(at 273.05 163.83 0)
 		(fields_autoplaced yes)
@@
 		)
 	)
-	(label "PWM6_DIR"
+	(label "PWM2_PWM"
 		(at 318.77 151.13 180)
 		(fields_autoplaced yes)
@@
 		)
 	)
-	(label "PWM7_STOP"
+	(label "PWM5_DIR"
 		(at 318.77 161.29 180)
 		(fields_autoplaced yes)
@@
 		)
 	)
-	(label "PWM9_PWM"
+	(label "PWM8_STOP"
 		(at 318.77 171.45 180)
 		(fields_autoplaced yes)
